Commit message: Change joint names

File: description/AROBO7.xacro (robot description, xacro)
@@ -342,5 +342,5 @@
   <child link="sprocket_new_v28_1_1"/>
 </joint>
-<joint name="Revolute 3" type="continuous">
+<joint name="Revolute_3" type="continuous">
   <origin xyz="-0.0185 0.029999 0.037" rpy="0 0 0"/>
   <parent link="drive_side_plate_v42_1_1"/>
@@ -353,5 +353,5 @@
   <child link="drive_side_plate_v42_Mirror__1_1"/>
 </joint>
-<joint name="Revolute 5" type="continuous">
+<joint name="Revolute_5" type="continuous">
   <origin xyz="0.0185 -0.026164 0.026162" rpy="0 0 0"/>
   <parent link="drive_side_plate_v42_Mirror__1_1"/>

File: description/robot.urdf.xacro (robot description, xacro)
@@ -1,5 +1,5 @@
 <?xml version="1.0"?>
 <robot xmlns:xacro="http://www.ros.org/wiki/xacro"  name="AROBO7">
-    <!-- Example link -->
     <xacro:include filename="AROBO7.xacro"/>
+    <xacro:include filename="gazebo_control.xacro"/>
 </robot>

Commit message: Add rviz launch file

File: description/AROBO7.xacro (robot description, xacro)
@@ -342,5 +342,5 @@
   <child link="sprocket_new_v28_1_1"/>
 </joint>
-<joint name="Revolute_3" type="continuous">
+<joint name="right_drive" type="continuous">
   <origin xyz="-0.0185 0.029999 0.037" rpy="0 0 0"/>
   <parent link="drive_side_plate_v42_1_1"/>
@@ -353,5 +353,5 @@
   <child link="drive_side_plate_v42_Mirror__1_1"/>
 </joint>
-<joint name="Revolute_5" type="continuous">
+<joint name="left_drive" type="continuous">
   <origin xyz="0.0185 -0.026164 0.026162" rpy="0 0 0"/>
   <parent link="drive_side_plate_v42_Mirror__1_1"/>

Commit message: Add LIDAR to gazebo

File: description/AROBO7.xacro (robot description, xacro)
@@ -232,24 +232,4 @@
   </collision>
 </link>
-<link name="rplidar_sensor_v1_1_1">
-  <inertial>
-    <origin xyz="-3.677012131997337e-07 -3.7389566448498e-07 0.00999977147532144" rpy="0 0 0"/>
-    <mass value="0.675231933814029"/>
-    <inertia ixx="0.000254" iyy="0.000254" izz="0.000462" ixy="-0.0" iyz="-0.0" ixz="-0.0"/>
-  </inertial>
-  <visual>
-    <origin xyz="-0.130894 -0.156967 -0.436527" rpy="0 0 0"/>
-    <geometry>
-      <mesh filename="package://AROBO7/description/meshes/rplidar_sensor_v1_1_1.stl" scale="0.001 0.001 0.001"/>
-    </geometry>
-    <material name="black"/>
-  </visual>
-  <collision>
-    <origin xyz="-0.130894 -0.156967 -0.436527" rpy="0 0 0"/>
-    <geometry>
-      <mesh filename="package://AROBO7/description/meshes/rplidar_sensor_v1_1_1.stl" scale="0.001 0.001 0.001"/>
-    </geometry>
-  </collision>
-</link>
 <link name="RpLidar_Case_Bot_v8_1_1">
   <inertial>
@@ -384,9 +364,4 @@
   <child link="RpLidar_Case_Top_High_v6_1_1"/>
 </joint>
-<joint name="Rigid 11" type="fixed">
-  <origin xyz="-0.0435 0.0 0.004" rpy="0 0 0"/>
-  <parent link="RpLidar_Case_Top_High_v6_1_1"/>
-  <child link="rplidar_sensor_v1_1_1"/>
-</joint>
 <joint name="Rigid 12" type="fixed">
   <origin xyz="0.062649 -0.04511 0.079821" rpy="0 0 0"/>

File: description/robot.urdf.xacro (robot description, xacro)
@@ -3,3 +3,4 @@
     <xacro:include filename="AROBO7.xacro"/>
     <xacro:include filename="gazebo_control.xacro"/>
+    <xacro:include filename="lidar.xacro"/>
 </robot>
