Commit message: Add command comments and finish camera joint

File: description/camera.xacro (robot description, xacro)
@@ -1,13 +1,20 @@
 <?xml version="1.0"?>
 <robot xmlns:xacro="http://www.ros.org/wiki/xacro" >
+<joint name="camera_joint" type="fixed">
+  <parent link="camera_front_v7_1_1"/>
+  <child link="camera_link"/>
+  <origin xyz="0 0 0" rpy="0 0 -1.57"/>
+</joint>
+<link name="camera_link">
+</link>
 <joint name="camera_optical_joint" type="fixed">
-  <parent link="camera_front_v7_1_1"/>
+  <parent link="camera_link"/>
   <child link="camera_link_optical"/>
   <origin xyz="0 0 0" rpy="0 0 0"/>
 </joint>
 <link name="camera_link_optical"></link>
-  <gazebo reference="camera_front_v7_1_1">
+  <gazebo reference="camera_link">
         <sensor name="camera" type="camera">
-            <pose> 0 0 0 -1.57 0 -1.57 </pose>
+            <pose> 0 0 0 0 0 0 </pose>
             <visualize>true</visualize>
             <update_rate>10</update_rate>
