Commit message: unbreak gazebo

File: description/robot.urdf.xacro (robot description, xacro)
@@ -1,7 +1,13 @@
 <?xml version="1.0"?>
 <robot xmlns:xacro="http://www.ros.org/wiki/xacro"  name="AROBO7">
+    <xacro:arg name="use_ros_2_control" default="true"/>
+    <xacro:arg name="sim_mode" default="true"/>
     <xacro:include filename="AROBO7.xacro"/>
-    <!-- <xacro:include filename="gazebo_control.xacro"/> -->
-    <xacro:include filename="ros2_control.xacro"/>
+    <xacro:if value="$(arg use_ros2_control)">
+        <xacro:include filename="ros2_control.xacro"/>
+    </xacro:if>
+    <xacro:unless value="$(arg use_ros2_control)">
+        <xacro:include filename="gazebo_control.xacro"/>
+    </xacro:unless>
     <xacro:include filename="lidar.xacro"/>
     <xacro:include filename="camera.xacro"/>

File: description/ros2_control.xacro (robot description, xacro)
@@ -1,4 +1,5 @@
 <?xml version="1.0"?>
 <robot xmlns:xacro="http://www.ros.org/wiki/xacro">
+<xacro:if value="$(arg sim_mode)">
     <ros2_control name="GazeboSystem" type="system">
         <hardware>
@@ -22,7 +23,39 @@
         </joint>
     </ros2_control>
+</xacro:if>
+<xacro:unless value="arg sim_mode">
+    <ros2_control name="RealRobot" type="system">
+        <hardware>
+            <plugin>diffdrive_arduino/DiffDriveArduino</plugin>
+            <param name="left_wheel_name">left_drive</param>
+            <param name="right_wheel_name">right_drive</param>
+            <param name="loop_rate">30</param>
+            <param name="device">/dev/serial/by-id/usb-FTDI_FT232R_USB_UART_B00055VV-if00-port0</param>
+            <param name="baud_rate">57600</param>
+            <param name="timeout">1000</param>
+            <param name="enc_counts_per_rev">2800</param>
+        </hardware>
+        <joint name="left_drive">
+            <command_interface name="velocity">
+                <param name="min">-10</param>
+                <param name="max">10</param>
+            </command_interface>
+            <state_interface name="velocity"></state_interface>
+            <state_interface name="position"></state_interface>
+        </joint>
+        <joint name="right_drive">
+            <command_interface name="velocity">
+                <param name="min">-10</param>
+                <param name="max">10</param>
+            </command_interface>
+            <state_interface name="velocity"></state_interface>
+            <state_interface name="position"></state_interface>
+        </joint>
+    </ros2_control>
+</xacro:unless>
     <gazebo>
         <plugin name="gazebo_ros2_control" filename="libgazebo_ros2_control.so">
             <parameters>$(find AROBO7)/config/my_controllers.yaml</parameters>
+            <parameters>$(find AROBO7)/config/gaz_ros2_ctl_use_sim.yaml</parameters>
         </plugin>
     </gazebo>

Commit message: make everything work again

File: description/robot.urdf.xacro (robot description, xacro)
@@ -2,8 +2,13 @@
 <robot xmlns:xacro="http://www.ros.org/wiki/xacro"  name="AROBO7">
     <xacro:arg name="use_ros_2_control" default="true"/>
-    <xacro:arg name="sim_mode" default="true"/>
+    <xacro:arg name="use_sim_mode" default="false"/>
     <xacro:include filename="AROBO7.xacro"/>
     <xacro:if value="$(arg use_ros2_control)">
-        <xacro:include filename="ros2_control.xacro"/>
+        <xacro:if value="$(arg use_sim_mode)">
+           <xacro:include filename="gazebo_ros2_control.xacro"/>
+        </xacro:if>
+        <xacro:unless value="$(arg use_sim_mode)">
+           <xacro:include filename="ros2_control.xacro"/>
+        </xacro:unless>
     </xacro:if>
     <xacro:unless value="$(arg use_ros2_control)">

File: description/ros2_control.xacro (robot description, xacro)
@@ -1,29 +1,6 @@
 <?xml version="1.0"?>
 <robot xmlns:xacro="http://www.ros.org/wiki/xacro">
-<!-- <xacro:if value="$(arg sim_mode)">
-    <ros2_control name="GazeboSystem" type="system">
-        <hardware>
-            <plugin>gazebo_ros2_control/GazeboSystem</plugin>
-        </hardware>
-        <joint name="left_drive">
-            <command_interface name="velocity">
-                <param name="min">-10</param>
-                <param name="max">10</param>
-            </command_interface>
-            <state_interface name="velocity"></state_interface>
-            <state_interface name="position"></state_interface>
-        </joint>
-        <joint name="right_drive">
-            <command_interface name="velocity">
-                <param name="min">-10</param>
-                <param name="max">10</param>
-            </command_interface>
-            <state_interface name="velocity"></state_interface>
-            <state_interface name="position"></state_interface>
-        </joint>
-    </ros2_control>
-</xacro:if> -->
-<!-- <xacro:unless value="arg sim_mode"> -->
-    <ros2_control name="RealRobot" type="system">
+    <!-- New code -->
+    <!-- <ros2_control name="RealRobot" type="system">
         <hardware>
             <plugin>diffdrive_arduino/DiffDriveArduinoHardware</plugin>
@@ -52,11 +29,33 @@
             <state_interface name="velocity"></state_interface>
         </joint>
+    </ros2_control> -->
+    <!-- Old code (just works) -->
+      <ros2_control name="RealRobot" type="system">
+        <hardware>
+            <plugin>diffdrive_arduino/DiffDriveArduino</plugin>
+            <param name="left_wheel_name">left_drive</param>
+            <param name="right_wheel_name">right_drive</param>
+            <param name="loop_rate">30</param>
+            <param name="device">/dev/serial/by-id/usb-FTDI_FT232R_USB_UART_B00055VV-if00-port0</param>
+            <param name="baud_rate">57600</param>
+            <param name="timeout">1000</param>
+            <param name="enc_counts_per_rev">2800</param>
+        </hardware>
+        <joint name="left_drive">
+            <command_interface name="velocity">
+                <param name="min">-10</param>
+                <param name="max">10</param>
+            </command_interface>
+            <state_interface name="velocity"></state_interface>
+            <state_interface name="position"></state_interface>
+        </joint>
+        <joint name="right_drive">
+            <command_interface name="velocity">
+                <param name="min">-10</param>
+                <param name="max">10</param>
+            </command_interface>
+            <state_interface name="velocity"></state_interface>
+            <state_interface name="position"></state_interface>
+        </joint>
     </ros2_control>
-<!-- </xacro:unless> -->
-    <gazebo>
-        <plugin name="gazebo_ros2_control" filename="libgazebo_ros2_control.so">
-            <parameters>$(find AROBO7)/config/my_controllers.yaml</parameters>
-            <parameters>$(find AROBO7)/config/gaz_ros2_ctl_use_sim.yaml</parameters>
-        </plugin>
-    </gazebo>
 </robot>
