Commit message: switch to arduiino UNO

File: description/ros2_control.xacro (robot description, xacro)
@@ -1,4 +1,34 @@
 <?xml version="1.0"?>
 <robot xmlns:xacro="http://www.ros.org/wiki/xacro">
+    <!-- Old code (just works) -->
+      <ros2_control name="RealRobot" type="system">
+        <hardware>
+            <plugin>diffdrive_arduino/DiffDriveArduino</plugin>
+            <param name="left_wheel_name">left_drive</param>
+            <param name="right_wheel_name">right_drive</param>
+            <param name="loop_rate">30</param>
+            <param name="device">/dev/serial/by-id/usb-Arduino__www.arduino.cc__0043_24238313935351818021-if00</param>
+            <param name="baud_rate">57600</param>
+            <param name="timeout">1000</param>
+            <param name="enc_counts_per_rev">2800</param>
+        </hardware>
+        <joint name="left_drive">
+            <command_interface name="velocity">
+                <param name="min">-10</param>
+                <param name="max">10</param>
+            </command_interface>
+            <state_interface name="velocity"></state_interface>
+            <state_interface name="position"></state_interface>
+        </joint>
+        <joint name="right_drive">
+            <command_interface name="velocity">
+                <param name="min">-10</param>
+                <param name="max">10</param>
+            </command_interface>
+            <state_interface name="velocity"></state_interface>
+            <state_interface name="position"></state_interface>
+        </joint>
+    </ros2_control>
+</robot>
     <!-- New code -->
     <!-- <ros2_control name="RealRobot" type="system">
@@ -30,32 +60,2 @@
         </joint>
     </ros2_control> -->
-    <!-- Old code (just works) -->
-      <ros2_control name="RealRobot" type="system">
-        <hardware>
-            <plugin>diffdrive_arduino/DiffDriveArduino</plugin>
-            <param name="left_wheel_name">left_drive</param>
-            <param name="right_wheel_name">right_drive</param>
-            <param name="loop_rate">30</param>
-            <param name="device">/dev/serial/by-id/usb-FTDI_FT232R_USB_UART_B00055VV-if00-port0</param>
-            <param name="baud_rate">57600</param>
-            <param name="timeout">1000</param>
-            <param name="enc_counts_per_rev">2800</param>
-        </hardware>
-        <joint name="left_drive">
-            <command_interface name="velocity">
-                <param name="min">-10</param>
-                <param name="max">10</param>
-            </command_interface>
-            <state_interface name="velocity"></state_interface>
-            <state_interface name="position"></state_interface>
-        </joint>
-        <joint name="right_drive">
-            <command_interface name="velocity">
-                <param name="min">-10</param>
-                <param name="max">10</param>
-            </command_interface>
-            <state_interface name="velocity"></state_interface>
-            <state_interface name="position"></state_interface>
-        </joint>
-    </ros2_control>
-</robot>
